File: pcb/pcb-v2-(using acheron setup)/_autosave-project.kicad_pcb (KiCad board)
At the start: 2 copper layers, 341 x 191.4 mm, 174 parts, among them J1 Conn_01x22_Female, J2 Conn_01x22_Male, J3 Conn_01x03_Male, J4 helios, SW1 CherryMX, SW10 CherryMX, SW11 CherryMX, SW12 CherryMX, SW13 CherryMX, SW14 CherryMX, SW15 CherryMX, SW16 CherryMX, SW17 CherryMX, SW18 CherryMX, SW19 CherryMX, SW2 CherryMX, SW20 CherryMX, SW21 CherryMX, SW22 CherryMX, SW23 CherryMX, SW24 CherryMX, SW25 CherryMX, SW26 CherryMX, SW27 CherryMX, SW28 CherryMX, SW29 CherryMX, SW3 CherryMX, SW30 CherryMX, SW31 CherryMX, SW32 CherryMX, SW33 CherryMX, SW34 CherryMX, SW35 CherryMX, SW36 CherryMX, SW37 CherryMX, SW38 CherryMX, SW39 CherryMX, SW4 CherryMX, SW40 CherryMX, SW41 CherryMX, SW42 CherryMX, SW43 CherryMX, SW44 CherryMX, SW45 CherryMX, SW46 CherryMX, SW47 CherryMX, SW48 CherryMX, SW49 CherryMX, SW5 CherryMX, SW50 CherryMX, SW51 CherryMX, SW52 CherryMX, SW53 CherryMX, SW54 CherryMX, SW55 CherryMX, SW56 CherryMX, SW57 CherryMX, SW58 CherryMX, SW59 CherryMX, SW6 CherryMX, SW60 CherryMX, SW61 CherryMX, SW62 CherryMX, SW63 CherryMX, SW64 CherryMX, SW65 CherryMX, SW66 CherryMX, SW67 CherryMX, SW68 CherryMX, SW69 CherryMX, SW7 CherryMX, SW70 CherryMX, SW71 CherryMX, SW72 CherryMX, SW73 CherryMX, SW74 CherryMX, SW75 CherryMX, SW76 CherryMX, SW77 CherryMX, SW78 CherryMX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

Commit message: added stuff
ik I am bad at commits so what whos gonna stop me *evil laughing*
Routing:
- net R6: track 357.6 -> 366.7 mm, vias 0 -> 1
- net Net-(D84-Pad2): track 0.00 -> 4.35 mm
- net Net-(D82-Pad2): track 0.00 -> 4.35 mm
- net Net-(D81-Pad2): track 0.00 -> 4.35 mm
- net Net-(D85-Pad2): track 0.00 -> 4.35 mm
- net Net-(D83-Pad2): track 0.00 -> 4.35 mm
- net Net-(D78-Pad2): track 0.00 -> 4.35 mm
- net Net-(D76-Pad2): track 0.00 -> 4.35 mm
- net Net-(D79-Pad2): track 0.00 -> 4.35 mm
- net Net-(SW77-Pad2): track 0.00 -> 4.35 mm
- net Net-(D72-Pad2): track 0.00 -> 4.35 mm
- net Net-(D70-Pad2): track 0.00 -> 4.35 mm
- net Net-(D74-Pad2): track 0.00 -> 4.35 mm
- net Net-(D73-Pad2): track 0.00 -> 4.35 mm
- net Net-(D71-Pad2): track 0.00 -> 4.35 mm
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Other:
- board size 341 x 191.4 mm -> 339.6 x 114.3 mm

Commit message: wiring added
Routing:
- net C8: track 0.00 -> 496.2 mm
- net C7: track 0.00 -> 494.3 mm
- net C6: track 0.00 -> 452.1 mm
- net C9: track 0.00 -> 448.0 mm
- net C5: track 0.00 -> 393.6 mm
- net C10: track 0.00 -> 391.4 mm
- net C4: track 0.00 -> 340.7 mm
- net C11: track 0.00 -> 333.8 mm
- net C12: track 0.00 -> 285.2 mm
- net C16: track 0.00 -> 255.3 mm
- net C13: track 0.00 -> 246.0 mm
- net C14: track 0.00 -> 243.2 mm
- net C15: track 0.00 -> 241.1 mm
- net C3: track 0.00 -> 165.1 mm
- net C2: track 0.00 -> 103.1 mm
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