File: pcb/pcb-v2-(using acheron setup)/project.kicad_pcb (KiCad board)
At the start: 2 copper layers, 339.6 x 114.3 mm, 174 parts, among them J1 Conn_01x22_Female, J2 Conn_01x22_Male, J3 Conn_01x03_Male, J4 helios, SW1 CherryMX, SW10 CherryMX, SW11 CherryMX, SW12 CherryMX, SW13 CherryMX, SW14 CherryMX, SW15 CherryMX, SW16 CherryMX, SW17 CherryMX, SW18 CherryMX, SW19 CherryMX, SW2 CherryMX, SW20 CherryMX, SW21 CherryMX, SW22 CherryMX, SW23 CherryMX, SW24 CherryMX, SW25 CherryMX, SW26 CherryMX, SW27 CherryMX, SW28 CherryMX, SW29 CherryMX, SW3 CherryMX, SW30 CherryMX, SW31 CherryMX, SW32 CherryMX, SW33 CherryMX, SW34 CherryMX, SW35 CherryMX, SW36 CherryMX, SW37 CherryMX, SW38 CherryMX, SW39 CherryMX, SW4 CherryMX, SW40 CherryMX, SW41 CherryMX, SW42 CherryMX, SW43 CherryMX, SW44 CherryMX, SW45 CherryMX, SW46 CherryMX, SW47 CherryMX, SW48 CherryMX, SW49 CherryMX, SW5 CherryMX, SW50 CherryMX, SW51 CherryMX, SW52 CherryMX, SW53 CherryMX, SW54 CherryMX, SW55 CherryMX, SW56 CherryMX, SW57 CherryMX, SW58 CherryMX, SW59 CherryMX, SW6 CherryMX, SW60 CherryMX, SW61 CherryMX, SW62 CherryMX, SW63 CherryMX, SW64 CherryMX, SW65 CherryMX, SW66 CherryMX, SW67 CherryMX, SW68 CherryMX, SW69 CherryMX, SW7 CherryMX, SW70 CherryMX, SW71 CherryMX, SW72 CherryMX, SW73 CherryMX, SW74 CherryMX, SW75 CherryMX, SW76 CherryMX, SW77 CherryMX, SW78 CherryMX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

Commit message: route but ima have to do a fucking nother gen of iterating ahahh
Routing:
- net C7: track 0.00 -> 500.2 mm
- net C8: track 0.00 -> 496.2 mm
- net C6: track 0.00 -> 452.1 mm
- net C9: track 0.00 -> 448.0 mm
- net C5: track 0.00 -> 393.6 mm
- net C10: track 0.00 -> 391.4 mm
- net C4: track 0.00 -> 340.9 mm
- net C11: track 0.00 -> 333.8 mm
- net C12: track 0.00 -> 285.2 mm
- net C3: track 0.00 -> 283.5 mm
- net C1: track 0.00 -> 263.0 mm
- net C16: track 0.00 -> 255.3 mm
- net C13: track 0.00 -> 246.0 mm
- net C2: track 0.00 -> 244.7 mm
- net C14: track 0.00 -> 243.2 mm
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
Commit message: routing v1 done and space bar stab added
Parts:
- SW36: footprint CherryMX:CherryMX_6.00u -> CherryMX_StabWireBottom:CherryMX_6.00u_StabWireBottom
Connections:
- J1 pad 1: R1 -> R6
- J1 pad 2: R2 -> R5
- J1 pad 3: R3 -> R4
- J1 pad 4: R4 -> R3
- J1 pad 5: R5 -> R2
- J1 pad 6: R6 -> R1
Routing:
- net R1: track 398.1 -> 648.0 mm, vias 0 -> 1
- net R2: track 396.2 -> 620.1 mm, vias 0 -> 1
- net R3: track 385.3 -> 578.9 mm, vias 0 -> 1
- net R4: track 380.4 -> 553.3 mm, vias 0 -> 1
- net R5: track 372.9 -> 465.6 mm, vias 0 -> 1
- net GP10: track 14.0 -> 69.8 mm
- net GP8: track 55.8 -> 0.00 mm
- net GP6: track 47.9 -> 0.00 mm
- net GP1: track 15.5 -> 63.4 mm
- net GP7: track 51.8 -> 68.1 mm
- net R6: track 366.7 -> 352.8 mm
- net C6: track 452.1 -> 465.0 mm
- net C5: track 393.6 -> 406.0 mm
- net GP21: track 11.7 -> 0.00 mm
- net GP23: track 14.2 -> 25.9 mm
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