File: pcb/pcb-v2-(using acheron setup)/project.kicad_pcb (KiCad board)
At the start: 2 copper layers, 337.4 x 114.3 mm, 174 parts, among them J1 Conn_01x22_Female, J2 Conn_01x22_Male, J3 Conn_01x03_Male, J4 helios, SW1 CherryMX, SW10 CherryMX, SW11 CherryMX, SW12 CherryMX, SW13 CherryMX, SW14 CherryMX, SW15 CherryMX, SW16 CherryMX, SW17 CherryMX, SW18 CherryMX, SW19 CherryMX, SW2 CherryMX, SW20 CherryMX, SW21 CherryMX, SW22 CherryMX, SW23 CherryMX, SW24 CherryMX, SW25 CherryMX, SW26 CherryMX, SW27 CherryMX, SW28 CherryMX, SW29 CherryMX, SW3 CherryMX, SW30 CherryMX, SW31 CherryMX, SW32 CherryMX, SW33 CherryMX, SW34 CherryMX, SW35 CherryMX, SW36 CherryMX, SW37 CherryMX, SW38 CherryMX, SW39 CherryMX, SW4 CherryMX, SW40 CherryMX, SW41 CherryMX, SW42 CherryMX, SW43 CherryMX, SW44 CherryMX, SW45 CherryMX, SW46 CherryMX, SW47 CherryMX, SW48 CherryMX, SW49 CherryMX, SW5 CherryMX, SW50 CherryMX, SW51 CherryMX, SW52 CherryMX, SW53 CherryMX, SW54 CherryMX, SW55 CherryMX, SW56 CherryMX, SW57 CherryMX, SW58 CherryMX, SW59 CherryMX, SW6 CherryMX, SW60 CherryMX, SW61 CherryMX, SW62 CherryMX, SW63 CherryMX, SW64 CherryMX, SW65 CherryMX, SW66 CherryMX, SW67 CherryMX, SW68 CherryMX, SW69 CherryMX, SW7 CherryMX, SW70 CherryMX, SW71 CherryMX, SW72 CherryMX, SW73 CherryMX, SW74 CherryMX, SW75 CherryMX, SW76 CherryMX, SW77 CherryMX, SW78 CherryMX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

Commit message: doneish?
Parts:
- removed J2: Conn_01x22_Male, Connector_FFC-FPC:Hirose_FH12-22S-0.5SH_1x22-1MP_P0.50mm_Horizontal
- removed J3: Conn_01x03_Male, Connector_PinSocket_1.27mm:PinSocket_1x03_P1.27mm_Vertical
- removed J4: helios, 0xCB-HeliosFootprint:helios
Routing:
- net GP25/RGB: track 79.4 -> 0.00 mm
- net GP8: track 55.8 -> 0.00 mm
- net GP7: track 51.8 -> 0.00 mm
- net GP6: track 47.9 -> 0.00 mm
- net GP5: track 38.9 -> 0.00 mm
- net 5V/RGB-Power: track 37.0 -> 0.00 mm
- net GND/RGB-GND: track 32.7 -> 0.00 mm
- net GP4: track 28.9 -> 0.00 mm
- net GP3: track 25.0 -> 0.00 mm
- net GP26: track 24.6 -> 0.00 mm
- net GP2: track 21.1 -> 0.00 mm
- net GP27: track 19.2 -> 0.00 mm
- net GP22: track 16.8 -> 0.00 mm
- net GP9: track 16.2 -> 0.00 mm
- net GP1: track 15.5 -> 0.00 mm
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Other:
- board size 337.4 x 114.3 mm -> 309.8 x 119.3 mm
- rule pad_to_mask_clearance: 0.1 -> 0
