File: pcb/pcb-v2-(using acheron setup)/project.kicad_sch (KiCad schematic)
At the start: 174 parts, among them J1 CherryMX, J2 Conn_01x22_Female, J3 Conn_01x22_Male, J4 Conn_01x03_Male, J5 helios, K1 CherryMX, M1 CherryMX, P1 CherryMX, Q1 CherryMX, T1 CherryMX, U1 CherryMX, X1 CherryMX, Y1 CherryMX

Commit message: added stuff
ik I am bad at commits so what whos gonna stop me *evil laughing*
Parts:
- renumbered D22 to D21, D23 to D22, D24 to D23, D25 to D24, D26 to D25, D27 to D26, D28 to D27, D29 to D28, D30 to D29, D31 to D30, D32 to D31, D33 to D32, D34 to D33, D35 to D34, D36 to D35, D37 to D36, D38 to D37, D39 to D38, D40 to D39, D41 to D40, D42 to D41, D43 to D42, D44 to D43, D45 to D44, D46 to D45, D47 to D46, D48 to D47, D49 to D48, D50 to D49, D51 to D50, D52 to D51, D53 to D52, D54 to D53, D55 to D54, D56 to D55, D57 to D56, D58 to D57, D59 to D58, D60 to D59, D61 to D60, D62 to D61, D63 to D62, D64 to D63, D65 to D64, D66 to D65, D67 to D66, D68 to D67, D69 to D68, D71 to D69, D72 to D70, D73 to D71, D74 to D72, D75 to D73, D70 to D74, D76 to D75, D77 to D76, D78 to D77, D79 to D78, D80 to D79, D81 to D80, D82 to D81, D83 to D82, D84 to D83, D85 to D84, D86 to D85, J2 to J1, J3 to J2, J4 to J3, J5 to J4, Escape1 to SW1, F2 to SW10, 2/@1 to SW11, Q1 to SW12, A1 to SW13, Z1 to SW14, Alt1 to SW15, F3 to SW16, 3/#1 to SW17, W1 to SW18, S1 to SW19, `/1 to SW2, X1 to SW20, F4 to SW21, 4/$1 to SW22, E1 to SW23, D21 to SW24, C1 to SW25, F5 to SW26, 5/%1 to SW27, R1 to SW28, F6 to SW29, Tab1 to SW3, V1 to SW30, F7 to SW31, 6/^1 to SW32, T1 to SW33, G1 to SW34, B1 to SW35, Space1 to SW36, F8 to SW37, 7/&1 to SW38, Y1 to SW39, CapLock1 to SW4, H1 to SW40, N1 to SW41, F9 to SW42, 8/*1 to SW43, U1 to SW44, J1 to SW45, M1 to SW46, F10 to SW47, 9/(1 to SW48, I1 to SW49, Ctrl1 to SW5, K1 to SW50, ,/<1 to SW51, F11 to SW52, 0/)1 to SW53, O1 to SW54, L1 to SW55, ./>1 to SW56, RAlt1 to SW57, F12 to SW58, -/_1 to SW59, F1 to SW6, P1 to SW60, ;/:1 to SW61, //1 to SW62, Super2 to SW63, F13 to SW64, =/+1 to SW65, [/{1 to SW66, '/"1 to SW67, Fn1 to SW68, PrtSc/Ins1 to SW69, 1/!1 to SW7, \/|1 to SW70, ]/}1 to SW71, Enter1 to SW72, RShift1 to SW73, LeftArrow1 to SW74, Pause/ScrLk1 to SW75, Macro1 to SW76, Backspace1 to SW77, UpArrow1 to SW78, DownArrow1 to SW79, LShift1 to SW8, Del1 to SW80, Home1 to SW81, PgUp1 to SW82, PgDn1 to SW83, End1 to SW84, RightArrow1 to SW85, Super1 to SW9
Other:
- moved on the sheet: D74

Commit message: draft routing complete now refining ig
Parts:
- SW36: footprint CherryMX:CherryMX_6.00u -> CherryMX_StabWireBottom:CherryMX_6.00u_StabWireBottom
Connections:
- net R1: now also J1.6 (Pin_6); no longer J1.1 (Pin_1)
- net R2: now also J1.5 (Pin_5); no longer J1.2 (Pin_2)
- net R3: now also J1.4 (Pin_4); no longer J1.3 (Pin_3)
- net R4: now also J1.3 (Pin_3); no longer J1.4 (Pin_4)
- net R5: now also J1.2 (Pin_2); no longer J1.5 (Pin_5)
- net R6: now also J1.1 (Pin_1); no longer J1.6 (Pin_6)
Changed lines of the file:
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@@
     )
   )
-  (global_label "R5" (shape input) (at 295.91 69.85 180) (fields_autoplaced)
+  (global_label "R5" (shape input) (at 295.91 62.23 180) (fields_autoplaced)
     (effects (font (size 1.27 1.27)) (justify right))
-    (property "Intersheet References" "${INTERSHEET_REFS}" (id 0) (at 291.0174 69.7706 0)
+    (property "Intersheet References" "${INTERSHEET_REFS}" (id 0) (at 291.0174 62.3094 0)
       (effects (font (size 1.27 1.27)) (justify right) hide)
     )
@@
     )
   )
-  (global_label "R2" (shape input) (at 295.91 62.23 180) (fields_autoplaced)
+  (global_label "R2" (shape input) (at 295.91 69.85 180) (fields_autoplaced)
     (effects (font (size 1.27 1.27)) (justify right))
-    (property "Intersheet References" "${INTERSHEET_REFS}" (id 0) (at 291.0174 62.1506 0)
+    (property "Intersheet References" "${INTERSHEET_REFS}" (id 0) (at 291.0174 69.9294 0)
       (effects (font (size 1.27 1.27)) (justify right) hide)
     )
@@
     )
   )
-  (global_label "R1" (shape input) (at 295.91 59.69 180) (fields_autoplaced)
+  (global_label "R1" (shape input) (at 295.91 72.39 180) (fields_autoplaced)
     (effects (font (size 1.27 1.27)) (justify right))
-    (property "Intersheet References" "${INTERSHEET_REFS}" (id 0) (at 291.0174 59.6106 0)
+    (property "Intersheet References" "${INTERSHEET_REFS}" (id 0) (at 291.0174 72.4694 0)
       (effects (font (size 1.27 1.27)) (justify right) hide)
     )
@@
     )
   )
-  (global_label "R3" (shape input) (at 295.91 64.77 180) (fields_autoplaced)
+  (global_label "R3" (shape input) (at 295.91 67.31 180) (fields_autoplaced)
     (effects (font (size 1.27 1.27)) (justify right))
-    (property "Intersheet References" "${INTERSHEET_REFS}" (id 0) (at 291.0174 64.6906 0)
+    (property "Intersheet References" "${INTERSHEET_REFS}" (id 0) (at 291.0174 67.3894 0)
       (effects (font (size 1.27 1.27)) (justify right) hide)
     )
@@
     )
   )
-  (global_label "R6" (shape input) (at 295.91 72.39 180) (fields_autoplaced)
+  (global_label "R6" (shape input) (at 295.91 59.69 180) (fields_autoplaced)
     (effects (font (size 1.27 1.27)) (justify right))
-    (property "Intersheet References" "${INTERSHEET_REFS}" (id 0) (at 291.0174 72.3106 0)
+    (property "Intersheet References" "${INTERSHEET_REFS}" (id 0) (at 291.0174 59.7694 0)
       (effects (font (size 1.27 1.27)) (justify right) hide)
     )
@@
     )
   )
-  (global_label "R4" (shape input) (at 295.91 67.31 180) (fields_autoplaced)
+  (global_label "R4" (shape input) (at 295.91 64.77 180) (fields_autoplaced)
     (effects (font (size 1.27 1.27)) (justify right))
-    (property "Intersheet References" "${INTERSHEET_REFS}" (id 0) (at 291.0174 67.2306 0)
+    (property "Intersheet References" "${INTERSHEET_REFS}" (id 0) (at 291.0174 64.8494 0)
       (effects (font (size 1.27 1.27)) (justify right) hide)
     )
@@
     (property "Reference" "SW36" (id 0) (at 116.84 119.38 0))
     (property "Value" "CherryMX" (id 1) (at 116.84 121.92 0))
-    (property "Footprint" "CherryMX:CherryMX_6.00u" (id 2) (at 116.84 126.365 0)
+    (property "Footprint" "CherryMX_StabWireBottom:CherryMX_6.00u_StabWireBottom" (id 2) (at 116.84 126.365 0)
       (effects (font (size 1.27 1.27)) hide)
     )
@@
     )
     (path "/5b501776-44a9-42cb-867a-253c7bce0f28"
-      (reference "SW36") (unit 1) (value "CherryMX") (footprint "CherryMX:CherryMX_6.00u")
+      (reference "SW36") (unit 1) (value "CherryMX") (footprint "CherryMX_StabWireBottom:CherryMX_6.00u_StabWireBottom")
     )
     (path "/76019206-3da3-478e-85c9-55c50424b5ff"
